Commit message: hector_quadrotor/hector_gazebo: converted gazebo plugins for 1.0

File: branches/fuerte/hector_models/hector_sensors_description/urdf/sonar_sensor.urdf.xacro (robot description, xacro)
@@ -51,5 +51,5 @@
           <updateRate>${update_rate}</updateRate>
           <topicName>${ros_topic}</topicName>
-          <frameId>/${name}_link</frameId>
+          <frameId>${name}_link</frameId>
         </controller:hector_gazebo_ros_sonar>
       </sensor:ray>

File: branches/fuerte/hector_quadrotor/hector_quadrotor_urdf/urdf/quadrotor_base.urdf.xacro (robot description, xacro)
@@ -53,24 +53,16 @@
         -->
         <topicName>cmd_vel</topicName>
-        <rollpitch>
-          <proportionalGain>10.0</proportionalGain>
-          <differentialGain>5.0</differentialGain>
-          <limit>0.5</limit>
-        </rollpitch>
-        <yaw>
-          <proportionalGain>2.0</proportionalGain>
-          <differentialGain>1.0</differentialGain>
-          <limit>1.5</limit>
-        </yaw>
-        <velocity_xy>
-          <proportionalGain>5.0</proportionalGain>
-          <differentialGain>1.0</differentialGain>
-          <limit>2</limit>
-        </velocity_xy>
-        <velocity_z>
-          <proportionalGain>5.0</proportionalGain>
-          <differentialGain>1.0</differentialGain>
-          <limit>2</limit>
-        </velocity_z>
+        <rollpitchProportionalGain>10.0</rollpitchProportionalGain>
+        <rollpitchDifferentialGain>5.0</rollpitchDifferentialGain>
+        <rollpitchLimit>0.5</rollpitchLimit>
+        <yawProportionalGain>2.0</yawProportionalGain>
+        <yawDifferentialGain>1.0</yawDifferentialGain>
+        <yawLimit>1.5</yawLimit>
+        <velocityXYProportionalGain>5.0</velocityXYProportionalGain>
+        <velocityXYDifferentialGain>1.0</velocityXYDifferentialGain>
+        <velocityXYLimit>2</velocityXYLimit>
+        <velocityZProportionalGain>5.0</velocityZProportionalGain>
+        <velocityZDifferentialGain>1.0</velocityZDifferentialGain>
+        <velocityZLimit>2</velocityZLimit>
         <maxForce>30</maxForce>
       </controller:hector_gazebo_quadrotor_simple_controller>
@@ -104,6 +96,6 @@
         <topicName>magnetic</topicName>
         <offset>0 0 0</offset>
-        <drift>0.1 0.1 0.1</drift>
-        <gaussianNoise>0.1 0.1 0.1</gaussianNoise>
+        <drift>0.01 0.01 0.01</drift>
+        <gaussianNoise>0.01 0.01 0.01</gaussianNoise>
       </controller:hector_gazebo_ros_magnetic>
       <controller:hector_gazebo_ros_gps name="quadrotor_gps_sim" plugin="libhector_gazebo_ros_gps.so">
