Commit message: [hector_ugv] -current state of fuerte migration (laser scanner and kinect geometry, textureless top box etc.)

File: branches/fuerte/hector_ugv_common/hector_ugv_description/urdf/hector_ugv.urdf.xacro (robot description, xacro)
@@ -11,5 +11,5 @@
   <include filename="$(find hector_ugv_description)/urdf/hector_ugv_base.urdf.xacro" />
   <hector_ugv_base wheel_joint_type="fixed" />
-  <include filename="$(find hector_ugv_description)/urdf/hector_ugv_openni_frames.urdf.xacro" />
+<!--  <include filename="$(find hector_ugv_description)/urdf/hector_ugv_openni_frames.urdf.xacro" />-->
   <include filename="$(find hector_sensors_description)/urdf/hokuyo_utm30lx.urdf.xacro" />
   <xacro:hokuyo_utm30lx name="laser1" parent="laser1_link" ros_topic="laser1/scan" update_rate="40" ray_count="1081" min_angle="135" max_angle="-135">

File: branches/fuerte/hector_ugv_common/hector_ugv_description/urdf/hector_ugv_base.urdf.xacro (robot description, xacro)
@@ -70,5 +70,5 @@
           <origin xyz="0.0 0.0 0.0" rpy="0 0 0" />
           <geometry>
-           <mesh filename="package://hector_ugv_description/meshes/$(env ROBOT)_top_box$(optenv TEST_SELF_FILTER).dae"/>
+           <mesh filename="package://hector_ugv_description/meshes/$(env ROBOT)_top_box$(optenv TEST_SELF_FILTER).stl"/>
           </geometry>
     </visual>
@@ -332,9 +332,9 @@
 <!--   <xacro:thermaleye_camera_model name="infrared" parent="mounting_link">
      <origin xyz="${infrared_x_position} ${infrared_y_position} ${infrared_z_position}" rpy="0 0 0" />
-   </xacro:thermaleye_camera_model>
+   </xacro:thermaleye_camera_model>-->
    <xacro:kinect_camera_model name="openni_camera" parent="mounting_link">
      <origin xyz="${kinect_x_position} 0 ${kinect_z_position}" rpy="0 0 0" />
    </xacro:kinect_camera_model>
-   <include filename="$(find monstertruck_urdf)/hector/$(env ROBOT)_addons.urdf.xacro" />-->
+   <include filename="$(find monstertruck_urdf)/hector/$(env ROBOT)_addons.urdf.xacro" />
   <hector_wheel parent="base_link" prefix="Front" suffix="left" reflect_x="1" reflect_y="1" wheel_joint_type="${wheel_joint_type}" />
   <hector_wheel parent="base_link" prefix="Front" suffix="right" reflect_x="1" reflect_y="-1" wheel_joint_type="${wheel_joint_type}" />

File: branches/fuerte/hector_ugv_common/hector_ugv_gazebo/urdf/hector_ugv.gazebo.xacro (robot description, xacro)
@@ -11,9 +11,9 @@
   <include filename="$(find hector_ugv_description)/urdf/hector_ugv_base.urdf.xacro" />
   <hector_ugv_base wheel_joint_type="continuous" />
-<!--  <include filename="$(find hector_sensors_description)/urdf/hokuyo_utm30lx.urdf.xacro" />
+  <include filename="$(find hector_sensors_description)/urdf/hokuyo_utm30lx.urdf.xacro" />
   <xacro:hokuyo_utm30lx name="laser1" parent="laser1_link" ros_topic="laser1/scan" update_rate="40" ray_count="1081" min_angle="135" max_angle="-135">
     <origin xyz="${laser1_center_x_offset} 0 ${laser1_plane_height}" rpy="0 0 0"/>
   </xacro:hokuyo_utm30lx>
-  <xacro:hokuyo_utm30lx name="laser0" parent="base_link" ros_topic="laser0/scan" update_rate="10" ray_count="700" min_angle="135" max_angle="-135">
+<!--  <xacro:hokuyo_utm30lx name="laser0" parent="base_link" ros_topic="laser0/scan" update_rate="10" ray_count="700" min_angle="135" max_angle="-135">
     <origin xyz="-0.18 0.0 0.173" rpy="0 ${-M_PI*0.5} 0" />
   </xacro:hokuyo_utm30lx>

Commit message: merged updates from trunk

File: branches/fuerte/hector_ugv_common/hector_ugv_description/urdf/hector_ugv.urdf.xacro (robot description, xacro)
@@ -8,11 +8,11 @@
   <include filename="$(find hector_ugv_description)/urdf/hector_wheel.urdf.xacro" />
   <include filename="$(find hector_ugv_description)/urdf/hector_ugv_common_dimensions.urdf.xacro" />
-  <include filename="$(find hector_ugv_description)/urdf/$(env ROBOT)_dimensions.urdf.xacro" />
+  <include filename="$(find hector_ugv_description)/urdf/hector1_dimensions.urdf.xacro" />
   <include filename="$(find hector_ugv_description)/urdf/hector_ugv_base.urdf.xacro" />
   <hector_ugv_base wheel_joint_type="fixed" />
-<!--  <include filename="$(find hector_ugv_description)/urdf/hector_ugv_openni_frames.urdf.xacro" />-->
+<!--  <include filename="$(find hector_ugv_description)/urdf/hector_ugv_openni_frames.urdf.xacro" />
   <include filename="$(find hector_sensors_description)/urdf/hokuyo_utm30lx.urdf.xacro" />
   <xacro:hokuyo_utm30lx name="laser1" parent="laser1_link" ros_topic="laser1/scan" update_rate="40" ray_count="1081" min_angle="135" max_angle="-135">
     <origin xyz="${laser1_center_x_offset} 0 ${laser1_plane_height}" rpy="0 0 0"/>
-  </xacro:hokuyo_utm30lx>
+  </xacro:hokuyo_utm30lx>-->
 </robot>

File: branches/fuerte/hector_ugv_common/hector_ugv_description/urdf/hector_ugv_base.urdf.xacro (robot description, xacro)
@@ -70,5 +70,5 @@
           <origin xyz="0.0 0.0 0.0" rpy="0 0 0" />
           <geometry>
-           <mesh filename="package://hector_ugv_description/meshes/$(env ROBOT)_top_box$(optenv TEST_SELF_FILTER).stl"/>
+           <mesh filename="package://hector_ugv_description/meshes/hector1_top_box$(optenv TEST_SELF_FILTER).dae"/>
           </geometry>
     </visual>
