Commit message: [fuerte/biorob_common] -merge changes from electric

File: branches/fuerte/biorob_common/biorob_description/urdf/biorob_v3_x4/biorob_v3_x4.urdf.xacro (robot description, xacro)
@@ -1,9 +1,9 @@
 <?xml version="1.0"?>
-<robot name="biorob_x4"
+<robot name="biorob_v3_x4"
     xmlns:sensor="http://playerstage.sourceforge.net/gazebo/xmlschema/#sensor"
     xmlns:controller="http://playerstage.sourceforge.net/gazebo/xmlschema/#controller"
     xmlns:interface="http://playerstage.sourceforge.net/gazebo/xmlschema/#interface">
     <!-- Included URDF Files -->
-    <include filename="$(find biorob_description)/urdf/biorob_x4/biorob_x4_base_self_filter.urdf.xacro" />
+    <include filename="$(find biorob_description)/urdf/biorob_v3_x4/biorob_v3_x4_base.urdf.xacro" />
     <link name="base">
       <inertial>
@@ -15,6 +15,6 @@
 	</inertial>
       </link>
-    <biorob_x4_arm parent="base" >
+    <biorob_v3_x4_arm parent="base" >
         <origin xyz="0 0 0" rpy="0 0 0"/>
-    </biorob_x4_arm>
+    </biorob_v3_x4_arm>
 </robot>

File: branches/fuerte/biorob_common/biorob_description/urdf/biorob_v3_x4/biorob_v3_x4_base.urdf.xacro (robot description, xacro)
@@ -1,12 +1,14 @@
 <?xml version="1.0"?>
-<robot xmlns:sensor="http://playerstage.sourceforge.net/gazebo/xmlschema/#sensor" xmlns:controller="http://playerstage.sourceforge.net/gazebo/xmlschema/#controller" xmlns:interface="http://playerstage.sourceforge.net/gazebo/xmlschema/#interface" xmlns:xacro="http://playerstage.sourceforge.net/gazebo/xmlschema/#interface" name="biorob_x4">
+<robot xmlns:sensor="http://playerstage.sourceforge.net/gazebo/xmlschema/#sensor"
+xmlns:controller="http://playerstage.sourceforge.net/gazebo/xmlschema/#controller"
+xmlns:interface="http://playerstage.sourceforge.net/gazebo/xmlschema/#interface"
+xmlns:xacro="http://playerstage.sourceforge.net/gazebo/xmlschema/#interface"
+name="biorob_v3_x4">
   <xacro:property name="base_height" value=".009"/>
   <xacro:property name="j1_length" value=".276"/>
   <!--0.285 to base plate-->
   <xacro:property name="j2_length" value=".307"/>
-  <xacro:property name="j3_length" value=".10"/>
-  <xacro:property name="j4_length" value=".209"/>
-  <xacro:property name="j5_length" value=".103"/>
-  <xacro:property name="j6_length" value=".021"/>
+  <xacro:property name="j3_length" value=".310"/>
+  <xacro:property name="j4_length" value=".103"/>
   <xacro:property name="pi" value="3.1415926536"/>
   <xacro:macro name="default_inertial" params="mass">
@@ -17,5 +19,5 @@
     </inertial>
   </xacro:macro>
-  <macro name="biorob_x4_arm" params="parent *origin">
+  <macro name="biorob_v3_x4_arm" params="parent *origin">
     <link name="biorob_base_link">
       <visual>
@@ -97,5 +99,5 @@
       <visual>
         <geometry>
-          <mesh filename="package://biorob_description/meshes/biorob_x6/biorob_x6_link_3.dae"/>
+          <mesh filename="package://biorob_description/meshes/biorob_common/biorob_link_3.dae"/>
           <!--<cylinder radius="0.02" length="${j3_length}" />-->
         </geometry>
@@ -106,5 +108,5 @@
       <collision>
         <geometry>
-          <mesh filename="package://biorob_description/meshes/biorob_x6/biorob_x6_link_3.dae"/>
+          <mesh filename="package://biorob_description/meshes/biorob_common/biorob_link_3.dae"/>
           <!--  <cylinder radius="0.02" length="${j3_length}" />-->
         </geometry>
@@ -121,6 +123,6 @@
       <visual>
         <geometry>
-          <mesh filename="package://biorob_description/meshes/biorob_x6/biorob_x6_link_4.dae"/>
-          <!--                    <cylinder radius="0.002" length="0.001" />-->
+          <mesh filename="package://biorob_description/meshes/biorob_common/biorob_link_4.dae"/>
+          <!--  <cylinder radius="0.02" length="${j4_length}" />-->
         </geometry>
         <origin xyz="0 0 0" rpy="${pi/2} 0 ${pi/2}"/>
@@ -130,28 +132,4 @@
       <collision>
         <geometry>
-          <mesh filename="package://biorob_description/meshes/biorob_x6/biorob_x6_link_4.dae"/>
-          <!--<cylinder radius="0.02" length="${j4_length}" />-->
-        </geometry>
-        <origin xyz="0 0 0" rpy="${pi/2} 0 ${pi/2}"/>
-      </collision>
-      <xacro:default_inertial mass="0.01"/>
-    </link>
-    <gazebo reference="biorob_link5">
-      <selfCollide>true</selfCollide>
-      <material>biorob_material/Grey</material>
-      <!--<material>HLUGV/Green</material>-->
-    </gazebo>
-    <link name="biorob_link5">
-      <visual>
-        <geometry>
-          <mesh filename="package://biorob_description/meshes/biorob_common/biorob_link_4.dae"/>
-          <!--  <cylinder radius="0.02" length="${j4_length}" />-->
-        </geometry>
-        <origin xyz="0 0 0" rpy="${pi/2} 0 ${pi/2}"/>
-        <material name="red">
-                </material>
-      </visual>
-      <collision>
-        <geometry>
           <mesh filename="package://biorob_description/meshes/biorob_common/biorob_link_4.dae"/>
           <!--<cylinder radius="0.02" length="${j4_length}" />-->
@@ -159,31 +137,7 @@
         <origin xyz="0 0 0" rpy="${pi/2} 0 ${pi/2}"/>
       </collision>
-      <xacro:default_inertial mass="0.01"/>
-    </link>
-    <gazebo reference="biorob_link5">
-      <selfCollide>true</selfCollide>
-      <material>biorob_material/Grey</material>
-      <!--<material>HLUGV/Green</material>-->
-    </gazebo>
-    <link name="biorob_link6">
-      <visual>
-        <geometry>
-          <mesh filename="package://biorob_description/meshes/biorob_x6/biorob_x6_link_6.dae"/>
-          <!--<cylinder radius="0.002" length="0.001" />-->
-        </geometry>
-        <origin xyz="0 0 0" rpy="${pi/2} 0 ${pi/2}"/>
-        <material name="red">
-                </material>
-      </visual>
-      <collision>
-        <geometry>
-          <mesh filename="package://biorob_description/meshes/biorob_x6/biorob_x6_link_6.dae"/>
-          <!--<cylinder radius="0.002" length="0.001" />-->
-        </geometry>
-        <origin xyz="0 0 0" rpy="${pi/2} 0 ${pi/2}"/>
-      </collision>
-      <xacro:default_inertial mass="0.01"/>
-    </link>
-    <gazebo reference="biorob_link6">
+      <xacro:default_inertial mass="0.1"/>
+    </link>
+    <gazebo reference="biorob_link4">
       <selfCollide>true</selfCollide>
       <material>biorob_material/Grey</material>
@@ -226,5 +180,5 @@
       <parent link="biorob_link3"/>
       <child link="biorob_link4"/>
-      <axis xyz="1 0 0"/>
+      <axis xyz="0 0 1"/>
       <origin xyz="${j3_length} 0 0.0"/>
       <limit effort="6.0" lower="${-pi*(100/180)}" upper="${pi*(100/180)}" velocity="1.5708"/>
@@ -232,27 +186,9 @@
       <dynamics damping="1.0" friction="1.0"/>
     </joint>
-    <joint name="joint5" type="revolute">
+    <joint name="tool_frame" type="fixed">
       <parent link="biorob_link4"/>
-      <child link="biorob_link5"/>
-      <axis xyz="0 0 1"/>
-      <origin xyz="${j4_length} 0 0.0"/>
-      <limit effort="6.0" lower="${-pi*(100/180)}" upper="${pi*(100/180)}" velocity="1.5708"/>
-      <!-- TODO: give correct effort limits -->
-      <dynamics damping="1.0" friction="1.0"/>
-    </joint>
-    <joint name="joint6" type="revolute">
-      <parent link="biorob_link5"/>
-      <child link="biorob_link6"/>
-      <axis xyz="1 0 0"/>
-      <origin xyz="${j5_length} 0.0 ${-j6_length} "/>
-      <limit effort="6.0" lower="${-pi*(100/180)}" upper="${pi*(100/180)}" velocity="1.5708"/>
-      <!-- TODO: give correct effort limits -->
-      <dynamics damping="1.0" friction="1.0"/>
-    </joint>
-    <joint name="tool_frame" type="fixed">
-      <parent link="biorob_link6"/>
       <child link="biorob_toolframe"/>
       <axis xyz="0 0 1"/>
-      <origin xyz="1 0.0 0.0" rpy="${-pi/2} 0 0"/>
+      <origin xyz="${j4_length} 0.0 0.0" rpy="${-pi/2} 0 0"/>
     </joint>
     <transmission type="pr2_mechanism_model/SimpleTransmission" name="joint1_trans">
@@ -276,15 +212,5 @@
       <mechanicalReduction>1.0</mechanicalReduction>
     </transmission>
-    <transmission type="pr2_mechanism_model/SimpleTransmission" name="joint5_trans">
-      <actuator name="joint5_motor"/>
-      <joint name="joint5"/>
-      <mechanicalReduction>1.0</mechanicalReduction>
-    </transmission>
-    <transmission type="pr2_mechanism_model/SimpleTransmission" name="joint6_trans">
-      <actuator name="joint6_motor"/>
-      <joint name="joint6"/>
-      <mechanicalReduction>1.0</mechanicalReduction>
-    </transmission>
-    <!--    <gazebo reference="biorob_toolframe">
+<!--    <gazebo reference="biorob_toolframe">
       <sensor:camera name="finger_tip_camera_sensor">
         <imageSize>640 480</imageSize>
@@ -299,17 +225,17 @@
           <imageTopicName>finger_tip_cam/image</imageTopicName>
           <frameName>biorob_toolframe</frameName>
-          <interface:camera name="finger_tip_camera_iface" />
+          <interface:camera name="finger_tip_camera_iface"/>
         </controller:gazebo_ros_camera>
       </sensor:camera>
       <turnGravityOff>true</turnGravityOff>
       <material>PR2/Blue</material>
+    </gazebo>
+    <gazebo>
+      <controller:gazebo_ros_controller_manager name="gazebo_ros_controller_manager" plugin="libgazebo_ros_controller_manager.so">
+        <alwaysOn>true</alwaysOn>
+        <updateRate>100.0</updateRate>
+        <interface:audio name="gazebo_ros_controller_manager_dummy_iface_biorob"/>
+      </controller:gazebo_ros_controller_manager>
     </gazebo>-->
-    <!--        <gazebo>
-              <controller:gazebo_ros_controller_manager name="gazebo_ros_controller_manager" plugin="libgazebo_ros_controller_manager.so">
-                <alwaysOn>true</alwaysOn>
-                <updateRate>100.0</updateRate>
-                <interface:audio name="gazebo_ros_controller_manager_dummy_iface_biorob" />
-              </controller:gazebo_ros_controller_manager>
-            </gazebo>-->
   </macro>
 </robot>

File: branches/fuerte/biorob_common/biorob_description/urdf/biorob_v3_x4/biorob_v3_x4_base_self_filter.urdf.xacro (robot description, xacro)
@@ -4,5 +4,5 @@
 xmlns:interface="http://playerstage.sourceforge.net/gazebo/xmlschema/#interface"
 xmlns:xacro="http://playerstage.sourceforge.net/gazebo/xmlschema/#interface"
-name="biorob_x4">
+name="biorob_v3_x4">
   <xacro:property name="base_height" value=".009"/>
   <xacro:property name="j1_length" value=".276"/>
@@ -19,5 +19,5 @@
     </inertial>
   </xacro:macro>
-  <macro name="biorob_x4_arm" params="parent *origin">
+  <macro name="biorob_v3_x4_arm" params="parent *origin">
     <link name="biorob_base_link">
       <visual>

File: branches/fuerte/biorob_common/biorob_description/urdf/biorob_v3_x4/biorob_v3_x4_self_filter.urdf.xacro (robot description, xacro)
@@ -1,9 +1,9 @@
 <?xml version="1.0"?>
-<robot name="biorob_x6"
+<robot name="biorob_v3_x4"
     xmlns:sensor="http://playerstage.sourceforge.net/gazebo/xmlschema/#sensor"
     xmlns:controller="http://playerstage.sourceforge.net/gazebo/xmlschema/#controller"
     xmlns:interface="http://playerstage.sourceforge.net/gazebo/xmlschema/#interface">
     <!-- Included URDF Files -->
-    <include filename="$(find biorob_description)/urdf/biorob_x6/biorob_x6_base.urdf.xacro" />
+    <include filename="$(find biorob_description)/urdf/biorob_x4/biorob_v3_x4_base_self_filter.urdf.xacro" />
     <link name="base">
       <inertial>
@@ -15,6 +15,6 @@
 	</inertial>
       </link>
-    <biorob_x4_arm parent="base" >
+    <biorob_v3_x4_arm parent="base" >
         <origin xyz="0 0 0" rpy="0 0 0"/>
-    </biorob_x4_arm>
+    </biorob_v3_x4_arm>
 </robot>

File: branches/fuerte/biorob_common/biorob_description/urdf/biorob_v3_x6/biorob_v3_x6.urdf.xacro (robot description, xacro)
@@ -1,9 +1,9 @@
 <?xml version="1.0"?>
-<robot name="biorob_x4"
+<robot name="biorob_v3_x6"
     xmlns:sensor="http://playerstage.sourceforge.net/gazebo/xmlschema/#sensor"
     xmlns:controller="http://playerstage.sourceforge.net/gazebo/xmlschema/#controller"
     xmlns:interface="http://playerstage.sourceforge.net/gazebo/xmlschema/#interface">
     <!-- Included URDF Files -->
-    <include filename="$(find biorob_description)/urdf/biorob_x4/biorob_x4_base.urdf.xacro" />
+    <include filename="$(find biorob_description)/urdf/biorob_v3_x6/biorob_v3_x6_base.urdf.xacro" />
     <link name="base">
       <inertial>
@@ -15,6 +15,6 @@
 	</inertial>
       </link>
-    <biorob_x4_arm parent="base" >
+    <biorob_v3_x6_arm parent="base" >
         <origin xyz="0 0 0" rpy="0 0 0"/>
-    </biorob_x4_arm>
+    </biorob_v3_x6_arm>
 </robot>

File: branches/fuerte/biorob_common/biorob_description/urdf/biorob_v3_x6/biorob_v3_x6_base.urdf.xacro (robot description, xacro)
@@ -1,14 +1,16 @@
 <?xml version="1.0"?>
 <robot xmlns:sensor="http://playerstage.sourceforge.net/gazebo/xmlschema/#sensor"
-xmlns:controller="http://playerstage.sourceforge.net/gazebo/xmlschema/#controller"
-xmlns:interface="http://playerstage.sourceforge.net/gazebo/xmlschema/#interface"
-xmlns:xacro="http://playerstage.sourceforge.net/gazebo/xmlschema/#interface"
-name="biorob_x4">
+       xmlns:controller="http://playerstage.sourceforge.net/gazebo/xmlschema/#controller"
+       xmlns:interface="http://playerstage.sourceforge.net/gazebo/xmlschema/#interface"
+       xmlns:xacro="http://playerstage.sourceforge.net/gazebo/xmlschema/#interface"
+       name="biorob_v3_x6">
   <xacro:property name="base_height" value=".009"/>
   <xacro:property name="j1_length" value=".276"/>
   <!--0.285 to base plate-->
   <xacro:property name="j2_length" value=".307"/>
-  <xacro:property name="j3_length" value=".310"/>
-  <xacro:property name="j4_length" value=".103"/>
+  <xacro:property name="j3_length" value=".10"/>
+  <xacro:property name="j4_length" value=".209"/>
+  <xacro:property name="j5_length" value=".103"/>
+  <xacro:property name="j6_length" value=".021"/>
   <xacro:property name="pi" value="3.1415926536"/>
   <xacro:macro name="default_inertial" params="mass">
@@ -19,5 +21,5 @@
     </inertial>
   </xacro:macro>
-  <macro name="biorob_x4_arm" params="parent *origin">
+  <macro name="biorob_v3_x6_arm" params="parent *origin">
     <link name="biorob_base_link">
       <visual>
@@ -99,5 +101,5 @@
       <visual>
         <geometry>
-          <mesh filename="package://biorob_description/meshes/biorob_common/biorob_link_3.dae"/>
+          <mesh filename="package://biorob_description/meshes/biorob_x6/biorob_v3_x6_link_3.dae"/>
           <!--<cylinder radius="0.02" length="${j3_length}" />-->
         </geometry>
@@ -108,5 +110,5 @@
       <collision>
         <geometry>
-          <mesh filename="package://biorob_description/meshes/biorob_common/biorob_link_3.dae"/>
+          <mesh filename="package://biorob_description/meshes/biorob_x6/biorob_v3_x6_link_3.dae"/>
           <!--  <cylinder radius="0.02" length="${j3_length}" />-->
         </geometry>
@@ -121,4 +123,28 @@
     </gazebo>
     <link name="biorob_link4">
+      <visual>
+        <geometry>
+          <mesh filename="package://biorob_description/meshes/biorob_x6/biorob_v3_x6_link_4.dae"/>
+          <!--                    <cylinder radius="0.002" length="0.001" />-->
+        </geometry>
+        <origin xyz="0 0 0" rpy="${pi/2} 0 ${pi/2}"/>
+        <material name="red">
+                </material>
+      </visual>
+      <collision>
+        <geometry>
+          <mesh filename="package://biorob_description/meshes/biorob_x6/biorob_v3_x6_link_4.dae"/>
+          <!--<cylinder radius="0.02" length="${j4_length}" />-->
+        </geometry>
+        <origin xyz="0 0 0" rpy="${pi/2} 0 ${pi/2}"/>
+      </collision>
+      <xacro:default_inertial mass="0.01"/>
+    </link>
+    <gazebo reference="biorob_link5">
+      <selfCollide>true</selfCollide>
+      <material>biorob_material/Grey</material>
+      <!--<material>HLUGV/Green</material>-->
+    </gazebo>
+    <link name="biorob_link5">
       <visual>
         <geometry>
@@ -137,7 +163,31 @@
         <origin xyz="0 0 0" rpy="${pi/2} 0 ${pi/2}"/>
       </collision>
-      <xacro:default_inertial mass="0.1"/>
-    </link>
-    <gazebo reference="biorob_link4">
+      <xacro:default_inertial mass="0.01"/>
+    </link>
+    <gazebo reference="biorob_link5">
+      <selfCollide>true</selfCollide>
+      <material>biorob_material/Grey</material>
+      <!--<material>HLUGV/Green</material>-->
+    </gazebo>
+    <link name="biorob_link6">
+      <visual>
+        <geometry>
+          <mesh filename="package://biorob_description/meshes/biorob_x6/biorob_v3_x6_link_6.dae"/>
+          <!--<cylinder radius="0.002" length="0.001" />-->
+        </geometry>
+        <origin xyz="0 0 0" rpy="${pi/2} 0 ${pi/2}"/>
+        <material name="red">
+                </material>
+      </visual>
+      <collision>
+        <geometry>
+          <mesh filename="package://biorob_description/meshes/biorob_x6/biorob_v3_x6_link_6.dae"/>
+          <!--<cylinder radius="0.002" length="0.001" />-->
+        </geometry>
+        <origin xyz="0 0 0" rpy="${pi/2} 0 ${pi/2}"/>
+      </collision>
+      <xacro:default_inertial mass="0.01"/>
+    </link>
+    <gazebo reference="biorob_link6">
       <selfCollide>true</selfCollide>
       <material>biorob_material/Grey</material>
@@ -180,5 +230,5 @@
       <parent link="biorob_link3"/>
       <child link="biorob_link4"/>
-      <axis xyz="0 0 1"/>
+      <axis xyz="1 0 0"/>
       <origin xyz="${j3_length} 0 0.0"/>
       <limit effort="6.0" lower="${-pi*(100/180)}" upper="${pi*(100/180)}" velocity="1.5708"/>
@@ -186,9 +236,27 @@
       <dynamics damping="1.0" friction="1.0"/>
     </joint>
+    <joint name="joint5" type="revolute">
+      <parent link="biorob_link4"/>
+      <child link="biorob_link5"/>
+      <axis xyz="0 0 1"/>
+      <origin xyz="${j4_length} 0 0.0"/>
+      <limit effort="6.0" lower="${-pi*(100/180)}" upper="${pi*(100/180)}" velocity="1.5708"/>
+      <!-- TODO: give correct effort limits -->
+      <dynamics damping="1.0" friction="1.0"/>
+    </joint>
+    <joint name="joint6" type="revolute">
+      <parent link="biorob_link5"/>
+      <child link="biorob_link6"/>
+      <axis xyz="1 0 0"/>
+      <origin xyz="${j5_length} 0.0 ${-j6_length} "/>
+      <limit effort="6.0" lower="${-pi*(100/180)}" upper="${pi*(100/180)}" velocity="1.5708"/>
+      <!-- TODO: give correct effort limits -->
+      <dynamics damping="1.0" friction="1.0"/>
+    </joint>
     <joint name="tool_frame" type="fixed">
-      <parent link="biorob_link4"/>
+      <parent link="biorob_link6"/>
       <child link="biorob_toolframe"/>
       <axis xyz="0 0 1"/>
-      <origin xyz="${j4_length} 0.0 0.0" rpy="${-pi/2} 0 0"/>
+      <origin xyz="1 0.0 0.0" rpy="${-pi/2} 0 0"/>
     </joint>
     <transmission type="pr2_mechanism_model/SimpleTransmission" name="joint1_trans">
@@ -212,5 +280,15 @@
       <mechanicalReduction>1.0</mechanicalReduction>
     </transmission>
-<!--    <gazebo reference="biorob_toolframe">
+    <transmission type="pr2_mechanism_model/SimpleTransmission" name="joint5_trans">
+      <actuator name="joint5_motor"/>
+      <joint name="joint5"/>
+      <mechanicalReduction>1.0</mechanicalReduction>
+    </transmission>
+    <transmission type="pr2_mechanism_model/SimpleTransmission" name="joint6_trans">
+      <actuator name="joint6_motor"/>
+      <joint name="joint6"/>
+      <mechanicalReduction>1.0</mechanicalReduction>
+    </transmission>
+    <!--    <gazebo reference="biorob_toolframe">
       <sensor:camera name="finger_tip_camera_sensor">
         <imageSize>640 480</imageSize>
@@ -225,17 +303,17 @@
           <imageTopicName>finger_tip_cam/image</imageTopicName>
           <frameName>biorob_toolframe</frameName>
-          <interface:camera name="finger_tip_camera_iface"/>
+          <interface:camera name="finger_tip_camera_iface" />
         </controller:gazebo_ros_camera>
       </sensor:camera>
       <turnGravityOff>true</turnGravityOff>
       <material>PR2/Blue</material>
-    </gazebo>
-    <gazebo>
-      <controller:gazebo_ros_controller_manager name="gazebo_ros_controller_manager" plugin="libgazebo_ros_controller_manager.so">
-        <alwaysOn>true</alwaysOn>
-        <updateRate>100.0</updateRate>
-        <interface:audio name="gazebo_ros_controller_manager_dummy_iface_biorob"/>
-      </controller:gazebo_ros_controller_manager>
     </gazebo>-->
+    <!--        <gazebo>
+              <controller:gazebo_ros_controller_manager name="gazebo_ros_controller_manager" plugin="libgazebo_ros_controller_manager.so">
+                <alwaysOn>true</alwaysOn>
+                <updateRate>100.0</updateRate>
+                <interface:audio name="gazebo_ros_controller_manager_dummy_iface_biorob" />
+              </controller:gazebo_ros_controller_manager>
+            </gazebo>-->
   </macro>
 </robot>

File: branches/fuerte/biorob_common/biorob_gazebo/urdf/biorob_v3_x4.gazebo.xacro (robot description, xacro)
@@ -1,8 +1,8 @@
 <?xml version="1.0"?>
-<robot name="biorob_x6"
+<robot name="biorob_v3_x4"
     xmlns:sensor="http://playerstage.sourceforge.net/gazebo/xmlschema/#sensor"
     xmlns:controller="http://playerstage.sourceforge.net/gazebo/xmlschema/#controller"
     xmlns:interface="http://playerstage.sourceforge.net/gazebo/xmlschema/#interface">
-  <include filename="$(find biorob_description)/urdf/biorob_x6/biorob_x6.urdf.xacro" />
+  <include filename="$(find biorob_description)/urdf/biorob_v3_x4/biorob_v3_x4.urdf.xacro" />
   <gazebo>
     <controller:gazebo_ros_controller_manager name="gazebo_ros_controller_manager" plugin="libgazebo_ros_controller_manager.so">

File: branches/fuerte/biorob_common/biorob_gazebo/urdf/biorob_v3_x6.gazebo.xacro (robot description, xacro)
@@ -1,8 +1,8 @@
 <?xml version="1.0"?>
-<robot name="biorob_x4"
+<robot name="biorob_v3_x6"
     xmlns:sensor="http://playerstage.sourceforge.net/gazebo/xmlschema/#sensor"
     xmlns:controller="http://playerstage.sourceforge.net/gazebo/xmlschema/#controller"
     xmlns:interface="http://playerstage.sourceforge.net/gazebo/xmlschema/#interface">
-  <include filename="$(find biorob_description)/urdf/biorob_x4/biorob_x4.urdf.xacro" />
+  <include filename="$(find biorob_description)/urdf/biorob_v3_x6/biorob_v3_x6.urdf.xacro" />
   <gazebo>
     <controller:gazebo_ros_controller_manager name="gazebo_ros_controller_manager" plugin="libgazebo_ros_controller_manager.so">
