Commit message: [fuerte/biorob_common] -merge changes from electric

File: branches/fuerte/biorob_common/biorob_description/urdf/biorob_ultra_x6/biorob_ultra_x6_base.urdf.xacro (robot description, xacro)
@@ -4,13 +4,13 @@
        xmlns:interface="http://playerstage.sourceforge.net/gazebo/xmlschema/#interface"
        xmlns:xacro="http://playerstage.sourceforge.net/gazebo/xmlschema/#interface"
-       name="biorob_v3_x6">
-  <xacro:property name="base_height" value=".009"/>
-  <xacro:property name="j1_length" value=".276"/>
+       name="biorob_ultra_x6">
+  <xacro:property name="base_height" value=".01"/>
+  <xacro:property name="j1_length" value=".284"/>
   <!--0.285 to base plate-->
-  <xacro:property name="j2_length" value=".307"/>
+  <xacro:property name="j2_length" value=".305"/>
   <xacro:property name="j3_length" value=".10"/>
-  <xacro:property name="j4_length" value=".209"/>
-  <xacro:property name="j5_length" value=".103"/>
-  <xacro:property name="j6_length" value=".021"/>
+  <xacro:property name="j4_length" value=".205"/>
+  <xacro:property name="j5_length" value=".14"/>
+  <xacro:property name="j6_length" value=".08"/>
   <xacro:property name="pi" value="3.1415926536"/>
   <xacro:macro name="default_inertial" params="mass">
@@ -21,5 +21,5 @@
     </inertial>
   </xacro:macro>
-  <macro name="biorob_v3_x6_arm" params="parent *origin">
+  <macro name="biorob_ultra_x6_arm" params="parent *origin">
     <link name="biorob_base_link">
       <visual>
@@ -173,5 +173,5 @@
       <visual>
         <geometry>
-          <mesh filename="package://biorob_description/meshes/biorob_x6/biorob_v3_x6_link_6.dae"/>
+          <mesh filename="package://biorob_description/meshes/biorob_ultra/biorob_ultra_tcp_end_80.dae"/>
           <!--<cylinder radius="0.002" length="0.001" />-->
         </geometry>
@@ -182,5 +182,5 @@
       <collision>
         <geometry>
-          <mesh filename="package://biorob_description/meshes/biorob_x6/biorob_v3_x6_link_6.dae"/>
+          <mesh filename="package://biorob_description/meshes/biorob_ultra/biorob_ultra_tcp_end_80.dae"/>
           <!--<cylinder radius="0.002" length="0.001" />-->
         </geometry>
@@ -249,5 +249,5 @@
       <child link="biorob_link6"/>
       <axis xyz="1 0 0"/>
-      <origin xyz="${j5_length} 0.0 ${-j6_length} "/>
+      <origin xyz="${j5_length} 0.0 0 "/>
       <limit effort="6.0" lower="${-pi*(100/180)}" upper="${pi*(100/180)}" velocity="1.5708"/>
       <!-- TODO: give correct effort limits -->
@@ -258,5 +258,5 @@
       <child link="biorob_toolframe"/>
       <axis xyz="0 0 1"/>
-      <origin xyz="0.02 0.0 0.0" rpy="${-pi/2} 0 0"/>
+      <origin xyz="${j6_length} 0.0 0.0" rpy="${-pi/2} 0 0"/>
     </joint>
     <transmission type="pr2_mechanism_model/SimpleTransmission" name="joint1_trans">
