Commit message: [biorob_description] -add proper model for ultra x5

File: branches/fuerte/biorob_common/biorob_description/urdf/biorob_ultra_x5/biorob_ultra_x5_base.urdf.xacro (robot description, xacro)
@@ -139,10 +139,10 @@
       <xacro:default_inertial mass="0.01"/>
     </link>-->
-    <gazebo reference="biorob_link5">
-      <selfCollide>true</selfCollide>
-      <material>biorob_material/Grey</material>
-      <!--<material>HLUGV/Green</material>-->
-    </gazebo>
-    <link name="biorob_link5">
+    <gazebo reference="biorob_link4">
+      <selfCollide>true</selfCollide>
+      <material>biorob_material/Grey</material>
+      <!--<material>HLUGV/Green</material>-->
+    </gazebo>
+    <link name="biorob_link4">
       <visual>
         <geometry>
@@ -163,10 +163,10 @@
       <xacro:default_inertial mass="0.01"/>
     </link>
-    <gazebo reference="biorob_link5">
-      <selfCollide>true</selfCollide>
-      <material>biorob_material/Grey</material>
-      <!--<material>HLUGV/Green</material>-->
-    </gazebo>
-    <link name="biorob_link6">
+    <gazebo reference="biorob_link4">
+      <selfCollide>true</selfCollide>
+      <material>biorob_material/Grey</material>
+      <!--<material>HLUGV/Green</material>-->
+    </gazebo>
+    <link name="biorob_link5">
       <visual>
         <geometry>
@@ -187,5 +187,5 @@
       <xacro:default_inertial mass="0.01"/>
     </link>
-    <gazebo reference="biorob_link6">
+    <gazebo reference="biorob_link5">
       <selfCollide>true</selfCollide>
       <material>biorob_material/Grey</material>
@@ -227,6 +227,6 @@
     <joint name="joint4" type="revolute">
       <parent link="biorob_link3"/>
-      <child link="biorob_link5"/>
-      <axis xyz="1 0 0"/>
+      <child link="biorob_link4"/>
+      <axis xyz="0 0 1"/>
       <origin xyz="${j3_length} 0 0.0"/>
       <limit effort="6.0" lower="${-pi*(100/180)}" upper="${pi*(100/180)}" velocity="1.5708"/>
@@ -242,7 +242,7 @@
       <dynamics damping="1.0" friction="1.0"/>
     </joint>-->
-    <joint name="joint6" type="revolute">
-      <parent link="biorob_link5"/>
-      <child link="biorob_link6"/>
+    <joint name="joint5" type="revolute">
+      <parent link="biorob_link4"/>
+      <child link="biorob_link5"/>
       <axis xyz="1 0 0"/>
       <origin xyz="${j5_length} 0.0 0 "/>
@@ -252,5 +252,5 @@
     </joint>
     <joint name="tool_frame" type="fixed">
-      <parent link="biorob_link6"/>
+      <parent link="biorob_link5"/>
       <child link="biorob_toolframe"/>
       <axis xyz="0 0 1"/>
