Commit message: [hlugv_common] -proper indendation for urdf parts

File: branches/fuerte/hlugv_common/hlugv_description/urdf/hlugv_base.urdf.xacro (robot description, xacro)
@@ -4,8 +4,4 @@
     xmlns:controller="http://playerstage.sourceforge.net/gazebo/xmlschema/#controller"
     xmlns:interface="http://playerstage.sourceforge.net/gazebo/xmlschema/#interface">
-    <!-- Included URDF Files -->
-    <!--<include filename="$(find erratic_description)/urdf/materials.urdf.xacro" />-->
-      <!--<include filename="$(find monstertruck_urdf)/hector/materials.urdf.xacro" />-->
-    <!--<include filename="$(find erratic_description)/urdf/erratic_computer.xacro" />-->
     <include filename="$(find hlugv_description)/urdf/hlugv_wheel.urdf.xacro" />
     <!-- Properties (Constants) -->
@@ -18,5 +14,5 @@
     <property name="wheel_size_y" value="0.05" />
     <property name="total_width" value="0.297" />
-<!--    <property name="wheel_offset_y" value="${(total_width - wheel_size_y) / 2}" />-->
+    <!--    <property name="wheel_offset_y" value="${(total_width - wheel_size_y) / 2}" />-->
     <property name="wheel_offset_y" value="0.12350" />
     <property name="wheel_offset_z_from_base_link" value="-0.029500" />
@@ -45,8 +41,8 @@
                 </geometry>
                 <material name="Green" >
-		        <color rgba="0 0.8 0 1"/>
+                    <color rgba="0 0.8 0 1"/>
                 </material>
             </visual>
-<!--            <collision>
+            <!--            <collision>
                 <origin xyz="0 0 ${base_size_z/2 + ground_clearance}" rpy="0 0 0" />
                 <geometry>
@@ -56,6 +52,4 @@
         </link>
         <joint name="base_footprint_joint" type="fixed">
-            <!-- NB: While you would think this would make it go up, it is oddly reversed.
-                 This moves the joint to 0,0,0 where we want it for rviz, etc. -->
             <origin xyz="0 0 ${base_size_z/2 + 0.051}" rpy="0 0 0" />
             <parent link="base_footprint"/>
@@ -75,7 +69,7 @@
                 <geometry>
                     <box size="${base_size_x} ${base_size_y} ${base_size_z}" />
-	      </geometry>
-              <material name="Grey" >
-		        <color rgba="0.8 0.8 0.8 1"/>
+                </geometry>
+                <material name="Grey" >
+                    <color rgba="0.8 0.8 0.8 1"/>
                 </material>
             </visual>
@@ -87,14 +81,13 @@
             </collision>
         </link>
-<!--	<hlugv_wheel suffix="left" parent="base_link" reflect="1"/>
-        <hlugv_wheel suffix="right" parent="base_link" reflect="-1"/>-->
-	<hlugv_wheel parent="base_link" prefix="front_left" offset_x= "0.15" offset_y = "${wheel_offset_y}" offset_z = "${wheel_offset_z_from_base_link}" reflect="1" />
-	<hlugv_wheel parent="base_link" prefix="mid_left" offset_x= "0.0" offset_y = "${wheel_offset_y}" offset_z = "${wheel_offset_z_from_base_link}" reflect="1" />
-	<hlugv_wheel parent="base_link" prefix="rear_left" offset_x= "-0.15" offset_y = "${wheel_offset_y}" offset_z = "${wheel_offset_z_from_base_link}" reflect="1" />
+        <!--	Add wheels using the hlugv_wheel macro -->
+        <hlugv_wheel parent="base_link" prefix="front_left" offset_x= "0.15" offset_y = "${wheel_offset_y}" offset_z = "${wheel_offset_z_from_base_link}" reflect="1" />
+        <hlugv_wheel parent="base_link" prefix="mid_left" offset_x= "0.0" offset_y = "${wheel_offset_y}" offset_z = "${wheel_offset_z_from_base_link}" reflect="1" />
+        <hlugv_wheel parent="base_link" prefix="rear_left" offset_x= "-0.15" offset_y = "${wheel_offset_y}" offset_z = "${wheel_offset_z_from_base_link}" reflect="1" />
         <hlugv_wheel parent="base_link" prefix="front_right" offset_x= "0.15" offset_y = "-${wheel_offset_y}" offset_z = "${wheel_offset_z_from_base_link}" reflect="1" />
-	<hlugv_wheel parent="base_link" prefix="mid_right" offset_x= "0.0" offset_y = "-${wheel_offset_y}" offset_z = "${wheel_offset_z_from_base_link}" reflect="1" />
-	<hlugv_wheel parent="base_link" prefix="rear_right" offset_x= "-0.15" offset_y = "-${wheel_offset_y}" offset_z = "${wheel_offset_z_from_base_link}" reflect="1" />
+        <hlugv_wheel parent="base_link" prefix="mid_right" offset_x= "0.0" offset_y = "-${wheel_offset_y}" offset_z = "${wheel_offset_z_from_base_link}" reflect="1" />
+        <hlugv_wheel parent="base_link" prefix="rear_right" offset_x= "-0.15" offset_y = "-${wheel_offset_y}" offset_z = "${wheel_offset_z_from_base_link}" reflect="1" />
         <gazebo>
-	    <controller:diffdrive_plugin_6w name="differential_drive_controller" plugin="libdiffdrive_plugin_6w.so">
+            <controller:diffdrive_plugin_6w name="differential_drive_controller" plugin="libdiffdrive_plugin_6w.so">
                 <alwaysOn>true</alwaysOn>
                 <update>100</update>
@@ -106,5 +99,5 @@
                 <rearLeftJoint>rear_left_wheel_joint</rearLeftJoint>
                 <rearRightJoint>rear_right_wheel_joint</rearRightJoint>
-               <wheelSeparation>${wheel_offset_y*2}</wheelSeparation>
+                <wheelSeparation>${wheel_offset_y*2}</wheelSeparation>
                 <wheelDiameter>${wheel_radius*2}</wheelDiameter>
                 <torque>5</torque>
@@ -113,58 +106,5 @@
                 <topicName>cmd_vel</topicName>
             </controller:diffdrive_plugin_6w>
-<!--            <controller:diffdrive_plugin_6w name="differential_drive_controller_1" plugin="libdiffdrive_plugin_6w.so">
-                <alwaysOn>true</alwaysOn>
-                <update>100</update>
-                <updateRate>100.0</updateRate>
-                <leftJoint>mid_right_wheel_joint</leftJoint>
-                <rightJoint>mid_left_wheel_joint</rightJoint>
-                <wheelSeparation>${wheel_offset_y*2}</wheelSeparation>
-                <wheelDiameter>${wheel_radius*2}</wheelDiameter>
-                <torque>5</torque>
-                <interface:position name="position_iface_0"/>
-                <robotNamespace>/</robotNamespace>
-                <topicName>cmd_vel</topicName>
-            </controller:diffdrive_plugin_6w>
-	    <controller:diffdrive_plugin_6w name="differential_drive_controller_2" plugin="libdiffdrive_plugin_6w.so">
-                <alwaysOn>true</alwaysOn>
-                <update>100</update>
-                <updateRate>100.0</updateRate>
-                <leftJoint>front_right_wheel_joint</leftJoint>
-                <rightJoint>front_left_wheel_joint</rightJoint>
-                <wheelSeparation>${wheel_offset_y*2}</wheelSeparation>
-                <wheelDiameter>${wheel_radius*2}</wheelDiameter>
-                <torque>5</torque>
-                <interface:position name="position_iface_1"/>
-                <robotNamespace>/</robotNamespace>
-                <topicName>cmd_vel</topicName>
-            </controller:diffdrive_plugin_6w>
-	    <controller:diffdrive_plugin_6w name="differential_drive_controller_3" plugin="libdiffdrive_plugin_6w.so">
-                <alwaysOn>true</alwaysOn>
-                <update>100</update>
-                <updateRate>100.0</updateRate>
-                <leftJoint>rear_right_wheel_joint</leftJoint>
-                <rightJoint>rear_left_wheel_joint</rightJoint>
-                <wheelSeparation>${wheel_offset_y*2}</wheelSeparation>
-                <wheelDiameter>${wheel_radius*2}</wheelDiameter>
-                <torque>5</torque>
-                <interface:position name="position_iface_2"/>
-                <robotNamespace>/</robotNamespace>
-                <topicName>cmd_vel</topicName>
-            </controller:diffdrive_plugin_6w>-->
-<!--            <controller:gazebo_ros_p3d name="p3d_base_controller" plugin="libgazebo_ros_p3d.so">
-                <alwaysOn>true</alwaysOn>
-                <updateRate>100.0</updateRate>
-                <bodyName>base_link</bodyName>
-                <topicName>base_pose_ground_truth</topicName>
-                <gaussianNoise>0.01</gaussianNoise>
-                <frameName>map</frameName>
-                <xyzOffsets>0 0 0</xyzOffsets>
-                <rpyOffsets>0 0 0</rpyOffsets>
-                <interface:position name="p3d_base_position"/>
-            </controller:gazebo_ros_p3d>-->
             <canonicalBody>base_footprint</canonicalBody>
-            <!-- this publishes empty joint_states due to no transmission, but
-             triggering robot_state_publisher to publish tf between fixed joints in erratic,
-             (e.g. base_laser_link for the base_scan frame) -->
             <controller:gazebo_ros_controller_manager name="gazebo_ros_controller_manager" plugin="libgazebo_ros_controller_manager.so">
                 <alwaysOn>true</alwaysOn>
@@ -172,5 +112,5 @@
                 <interface:audio name="gazebo_ros_controller_manager_dummy_iface" />
             </controller:gazebo_ros_controller_manager>
-	    <controller:gazebo_ros_imu name="imu_controller" plugin="libgazebo_ros_imu.so">
+            <controller:gazebo_ros_imu name="imu_controller" plugin="libgazebo_ros_imu.so">
                 <alwaysOn>true</alwaysOn>
                 <updateRate>50</updateRate>
@@ -183,9 +123,9 @@
             </controller:gazebo_ros_imu>
         </gazebo>
-	<gazebo reference="base_link">
-           <material>HLUGV/Green</material>
+        <gazebo reference="base_link">
+            <material>HLUGV/Green</material>
         </gazebo>
-	<gazebo reference="base_link">
-           <material>HLUGV/Green</material>
+        <gazebo reference="base_link">
+            <material>HLUGV/Green</material>
         </gazebo>
     </macro>

File: branches/fuerte/hlugv_common/hlugv_description/urdf/hlugv_wheel.urdf.xacro (robot description, xacro)
@@ -5,71 +5,61 @@
     xmlns:interface="http://playerstage.sourceforge.net/gazebo/xmlschema/#interface"
 	  xmlns:xacro="http://playerstage.sourceforge.net/gazebo/xmlschema/#interface">
-  <!-- Properties (Constants) -->
-  <xacro:property name="M_PI" value="3.14159" />
-  <xacro:property name="wheel_radius" value="0.063" />
-  <xacro:property name="wheel_size_y" value="0.05" />
-  <xacro:property name="wheel_offset_x" value="0.16" />
-  <xacro:property name="wheel_offset_y" value="0.155" /> <!-- half of wheel width + half of socket width + gap -->
-  <xacro:property name="wheel_offset_z" value="-0.112" /> <!-- wheel_radius - socket height -->
-  <xacro:macro name="hlugv_wheel" params="parent prefix offset_x offset_y offset_z reflect">
-    <joint name="${prefix}_wheel_joint" type="continuous">
-      <origin xyz="${offset_x } ${offset_y * reflect} ${offset_z}" rpy="0 0 0" />
-      <parent link="${parent}" />
-      <child link="${prefix}_wheel_link" />
-      <axis xyz="0 1 0" />
-      <limit effort="100" velocity="100" />
-      <joint_properties damping="0.0" friction="0.0" />
-      <anchor xyz="0 0 0" />
-      <!--<mimic joint="steer${prefix}" multiplier="1.234" offset="0.0" />-->
-    </joint>
-<!--    <joint name="${prefix}_${suffix}_motor_joint" type="fixed">
-      <origin xyz="${wheel_offset_x * reflect_x} ${wheel_offset_y * reflect_y} ${wheel_offset_z}" rpy="0 0 0" />
-      <parent link="${parent}" />
-      <child link="${prefix}_${suffix}_motor_link" />
-    </joint> -->
-    <link name="${prefix}_wheel_link">
-      <inertial>
-        <mass value="0.1" />
-        <origin xyz=" 0 0 0 " />
+    <!-- Properties (Constants) -->
+    <xacro:property name="M_PI" value="3.14159" />
+    <xacro:property name="wheel_radius" value="0.063" />
+    <xacro:property name="wheel_size_y" value="0.05" />
+    <xacro:property name="wheel_offset_x" value="0.16" />
+    <xacro:property name="wheel_offset_y" value="0.155" />
+     <!-- half of wheel width + half of socket width + gap -->
+    <xacro:property name="wheel_offset_z" value="-0.112" />
+     <!-- wheel_radius - socket height -->
+    <xacro:macro name="hlugv_wheel" params="parent prefix offset_x offset_y offset_z reflect">
+        <joint name="${prefix}_wheel_joint" type="continuous">
+            <origin xyz="${offset_x } ${offset_y * reflect} ${offset_z}" rpy="0 0 0" />
+            <parent link="${parent}" />
+            <child link="${prefix}_wheel_link" />
+            <axis xyz="0 1 0" />
+            <limit effort="100" velocity="100" />
+            <joint_properties damping="0.0" friction="0.0" />
+            <anchor xyz="0 0 0" />
+        </joint>
+        <link name="${prefix}_wheel_link">
+            <inertial>
+                <mass value="0.1" />
+                <origin xyz=" 0 0 0 " />
                 <inertia  ixx="0.00012411765597" ixy="0.0" ixz="0.0"
                           iyy="0.00015218160428" iyz="0.0"
                           izz="0.00011763977943" />
-      </inertial>
-      <visual>
-        <origin xyz="0 0 0" rpy="${-M_PI/2} 0 0" />
-        <geometry>
-          <cylinder radius="${wheel_radius}" length="${wheel_size_y}"/>
-        </geometry>
-                      <material name="DarkGrey" >
-		        <color rgba="0.3 0.3 0.3 1"/>
+            </inertial>
+            <visual>
+                <origin xyz="0 0 0" rpy="${-M_PI/2} 0 0" />
+                <geometry>
+                    <cylinder radius="${wheel_radius}" length="${wheel_size_y}"/>
+                </geometry>
+                <material name="DarkGrey" >
+                    <color rgba="0.3 0.3 0.3 1"/>
                 </material>
-      </visual>
-      <collision>
-        <origin xyz="0 0 0" rpy="${-M_PI/2} 0 0" />
-        <geometry>
-          <cylinder radius="${wheel_radius}" length="${wheel_size_y}" />
-        </geometry>
-        <material name="MTWheelColMat"/>
-      </collision>
-    </link>
-    <gazebo reference="${prefix}_wheel_link" >
-      <mu1 value="100.0" />
-      <mu2 value="100.0" />
-      <kp  value="100000.0" />
-      <kd  value="1.0" />
-      <material>HLUGV/Grey</material>
-    </gazebo>
-    <transmission type="pr2_mechanism_model/SimpleTransmission" name="${prefix}_wheel_trans">
-      <actuator name="${prefix}_motor_link" />
-      <joint name="${prefix}_wheel_joint" />
-      <mechanicalReduction>1.0</mechanicalReduction>
-      <motorTorqueConstant>1</motorTorqueConstant>
-    </transmission>
-<!--    <transmission type="pr2_mechanism_model/SimpleTransmission" name="${prefix}_${suffix}_steering_trans">
-      <actuator name="${parent}" />
-      <joint name="${prefix}_${suffix}_steering_joint" />
-      <mechanicalReduction>${reflect_x}</mechanicalReduction>
-      <motorTorqueConstant>1</motorTorqueConstant>
-    </transmission>-->
-  </xacro:macro>
+            </visual>
+            <collision>
+                <origin xyz="0 0 0" rpy="${-M_PI/2} 0 0" />
+                <geometry>
+                    <cylinder radius="${wheel_radius}" length="${wheel_size_y}" />
+                </geometry>
+                <material name="MTWheelColMat"/>
+            </collision>
+        </link>
+        <gazebo reference="${prefix}_wheel_link" >
+            <mu1 value="100.0" />
+            <mu2 value="100.0" />
+            <kp  value="100000.0" />
+            <kd  value="1.0" />
+            <material>HLUGV/Grey</material>
+        </gazebo>
+        <transmission type="pr2_mechanism_model/SimpleTransmission" name="${prefix}_wheel_trans">
+            <actuator name="${prefix}_motor_link" />
+            <joint name="${prefix}_wheel_joint" />
+            <mechanicalReduction>1.0</mechanicalReduction>
+            <motorTorqueConstant>1</motorTorqueConstant>
+        </transmission>
+    </xacro:macro>
 </robot>
