Commit message: merged updates from /fuerte/trunk

File: electric/trunk/hector_quadrotor/hector_quadrotor_controller/urdf/quadrotor_propulsion.urdf.xacro (robot description, xacro)
@@ -5,11 +5,13 @@
 >
   <!-- Quadrotor Aerodynamics Plugin -->
-  <xacro:macro name="quadrotor_aerodynamics">
+  <xacro:macro name="quadrotor_propulsion">
     <gazebo>
-      <controller:hector_gazebo_quadrotor_aerodynamics name="quadrotor_aerodynamics" plugin="libhector_gazebo_quadrotor_aerodynamics.so">
+      <controller:hector_gazebo_quadrotor_propulsion name="quadrotor_propulsion" plugin="libhector_gazebo_quadrotor_propulsion.so">
         <alwaysOn>true</alwaysOn>
         <updateRate>0.0</updateRate>
         <bodyName>base_link</bodyName>
-      </controller:hector_gazebo_quadrotor_aerodynamics>
+        <controlRate>100.0</controlRate>
+        <controlDelay>0.01</controlDelay>
+      </controller:hector_gazebo_quadrotor_propulsion>
     </gazebo>
   </xacro:macro>

File: electric/trunk/hector_quadrotor/hector_quadrotor_controller/urdf/quadrotor_simple_controller.urdf.xacro (robot description, xacro)
@@ -5,5 +5,5 @@
 >
   <!-- Quadrotor Simple Controller Plugin -->
-  <xacro:macro name="quadrotor_controller">
+  <xacro:macro name="quadrotor_simple_controller">
     <gazebo>
       <controller:hector_gazebo_quadrotor_simple_controller name="quadrotor_simple_controller" plugin="libhector_gazebo_quadrotor_simple_controller.so">
