Commit message: [biorob_description] added toolframe geometry to display it in rviz / updated coordinate systems to be consistent to dh-description

File: fuerte/trunk/biorob_common/biorob_description/urdf/biorob_ultra_x4/biorob_ultra_x4_base.urdf.xacro (robot description, xacro)
@@ -77,5 +77,5 @@
         </geometry>
         <!--<origin xyz="${j2_length/2 - j2_overhang_rear/2 } 0 0" rpy="0 ${pi/2} 0"/>-->
-        <origin xyz="0 0 0" rpy="${-pi/2} ${pi/2} 0"/>
+        <origin xyz="0 0 0" rpy="0 ${pi/2} ${pi}"/>
         <material name="red">
           <color rgba="0.6 0.6 0.6 1"/>
@@ -87,5 +87,5 @@
           <!--<cylinder radius="0.02" length="${j2_length}" />-->
         </geometry>
-        <origin xyz="0 0 0" rpy="${-pi/2} ${pi/2} 0"/>
+        <origin xyz="0 0 0" rpy="0 ${pi/2} ${pi}"/>
       </collision>
       <xacro:default_inertial mass="0.5"/>
@@ -145,4 +145,18 @@
     </gazebo>
     <link name="biorob_toolframe">
+      <visual>
+        <geometry>
+          <cylinder radius="0.01" length="0.001" />
+        </geometry>
+        <origin xyz="0 0 0" rpy="${pi/2} 0 ${pi/2}"/>
+        <material name="red">
+        </material>
+      </visual>
+      <collision>
+        <geometry>
+          <cylinder radius="0.02" length="0.001" />
+        </geometry>
+        <origin xyz="0 0 0" rpy="${pi/2} 0 ${pi/2}"/>
+      </collision>
       <xacro:default_inertial mass="0.05"/>
     </link>
@@ -165,5 +179,5 @@
       <child link="biorob_link2"/>
       <axis xyz="0 0 1"/>
-      <origin xyz="0 0 ${j1_length-base_height}" rpy="${pi/2} -${pi/2} 0"/>
+      <origin xyz="0 0 ${j1_length-base_height}" rpy="${pi/2} 0 0"/>
       <limit effort="6.0" lower="${-pi*(170/180)}" upper="${pi*(170/180)}" velocity="1.5708"/>
       <dynamics damping="1.0" friction="1.0"/>
@@ -173,5 +187,5 @@
       <child link="biorob_link3"/>
       <axis xyz="0 0 1 "/>
-      <origin xyz="${j2_length} 0 0.0"/>
+      <origin xyz="0 ${j2_length} 0" rpy="0 0 ${pi/2}"/>
       <limit effort="6.0" lower="${-pi*(100/180)}" upper="${pi*(100/180)}" velocity="1.5708"/>
       <dynamics damping="1.0" friction="1.0"/>
@@ -190,5 +204,5 @@
       <child link="biorob_toolframe"/>
       <axis xyz="0 0 1"/>
-      <origin xyz="${j4_length} 0.0 0.0" rpy="${-pi/2} 0 0"/>
+      <origin xyz="${j4_length} 0.0 0.0" rpy="0 0 0"/>
     </joint>
     <transmission type="pr2_mechanism_model/SimpleTransmission" name="joint1_trans">

File: fuerte/trunk/biorob_common/biorob_description/urdf/biorob_ultra_x4_hp/biorob_ultra_x4_hp_base.urdf.xacro (robot description, xacro)
@@ -77,5 +77,5 @@
         </geometry>
         <!--<origin xyz="${j2_length/2 - j2_overhang_rear/2 } 0 0" rpy="0 ${pi/2} 0"/>-->
-        <origin xyz="0 0 0" rpy="${-pi/2} ${pi/2} 0"/>
+        <origin xyz="0 0 0" rpy="0 ${pi/2} ${pi}"/>
         <material name="red">
           <color rgba="0.6 0.6 0.6 1"/>
@@ -87,5 +87,5 @@
           <!--<cylinder radius="0.02" length="${j2_length}" />-->
         </geometry>
-        <origin xyz="0 0 0" rpy="${-pi/2} ${pi/2} 0"/>
+        <origin xyz="0 0 0" rpy="0 ${pi/2} ${pi}"/>
       </collision>
       <xacro:default_inertial mass="0.5"/>
@@ -145,4 +145,18 @@
     </gazebo>
     <link name="biorob_toolframe">
+      <visual>
+        <geometry>
+          <cylinder radius="0.01" length="0.001" />
+        </geometry>
+        <origin xyz="0 0 0" rpy="${pi/2} 0 ${pi/2}"/>
+        <material name="red">
+        </material>
+      </visual>
+      <collision>
+        <geometry>
+          <cylinder radius="0.02" length="0.001" />
+        </geometry>
+        <origin xyz="0 0 0" rpy="${pi/2} 0 ${pi/2}"/>
+      </collision>
       <xacro:default_inertial mass="0.05"/>
     </link>
@@ -165,5 +179,5 @@
       <child link="biorob_link2"/>
       <axis xyz="0 0 1"/>
-      <origin xyz="0 0 ${j1_length-base_height}" rpy="${pi/2} -${pi/2} 0"/>
+      <origin xyz="0 0 ${j1_length-base_height}" rpy="${pi/2} 0 0"/>
       <limit effort="6.0" lower="${-pi*(170/180)}" upper="${pi*(170/180)}" velocity="1.5708"/>
       <dynamics damping="1.0" friction="1.0"/>
@@ -173,5 +187,5 @@
       <child link="biorob_link3"/>
       <axis xyz="0 0 1 "/>
-      <origin xyz="${j2_length} 0 0.0"/>
+      <origin xyz="0 ${j2_length} 0" rpy="0 0 ${pi/2}"/>
       <limit effort="6.0" lower="${-pi*(100/180)}" upper="${pi*(100/180)}" velocity="1.5708"/>
       <dynamics damping="1.0" friction="1.0"/>
@@ -190,5 +204,5 @@
       <child link="biorob_toolframe"/>
       <axis xyz="0 0 1"/>
-      <origin xyz="${j4_length} 0.0 0.0" rpy="${-pi/2} 0 0"/>
+      <origin xyz="${j4_length} 0.0 0.0" rpy="0 0 0"/>
     </joint>
     <transmission type="pr2_mechanism_model/SimpleTransmission" name="joint1_trans">

File: fuerte/trunk/biorob_common/biorob_description/urdf/biorob_ultra_x5_hg/biorob_ultra_x5_hg_base.urdf.xacro (robot description, xacro)
@@ -79,5 +79,5 @@
         </geometry>
         <!--<origin xyz="${j2_length/2 - j2_overhang_rear/2 } 0 0" rpy="0 ${pi/2} 0"/>-->
-        <origin xyz="0 0 0" rpy="${-pi/2} ${pi/2} 0"/>
+        <origin xyz="0 0 0" rpy="0 ${pi/2} ${pi}"/>
         <material name="red">
           <color rgba="0.6 0.6 0.6 1"/>
@@ -89,5 +89,5 @@
           <!--<cylinder radius="0.02" length="${j2_length}" />-->
         </geometry>
-        <origin xyz="0 0 0" rpy="${-pi/2} ${pi/2} 0"/>
+        <origin xyz="0 0 0" rpy="0 ${pi/2} ${pi}"/>
       </collision>
       <xacro:default_inertial mass="0.5"/>
@@ -174,5 +174,5 @@
           <!--<cylinder radius="0.002" length="0.001" />-->
         </geometry>
-        <origin xyz="0 0 0" rpy="${pi/2} 0 ${pi/2}"/>
+        <origin xyz="0 0 0" rpy="0 0 0"/>
         <material name="red">
                 </material>
@@ -183,5 +183,5 @@
           <!--<cylinder radius="0.002" length="0.001" />-->
         </geometry>
-        <origin xyz="0 0 0" rpy="${pi/2} 0 ${pi/2}"/>
+        <origin xyz="0 0 0" rpy="0 0 0"/>
       </collision>
       <xacro:default_inertial mass="0.01"/>
@@ -193,4 +193,18 @@
     </gazebo>
     <link name="biorob_toolframe">
+      <visual>
+        <geometry>
+          <cylinder radius="0.01" length="0.001" />
+        </geometry>
+        <origin xyz="0 0 0" rpy="0 0 0"/>
+        <material name="red">
+        </material>
+      </visual>
+      <collision>
+        <geometry>
+          <cylinder radius="0.01" length="0.001" />
+        </geometry>
+        <origin xyz="0 0 0" rpy="0 0 0"/>
+      </collision>
       <xacro:default_inertial mass="0.05"/>
     </link>
@@ -213,5 +227,5 @@
       <child link="biorob_link2"/>
       <axis xyz="0 0 1"/>
-      <origin xyz="0 0 ${j1_length-base_height}" rpy="${pi/2} -${pi/2} 0"/>
+      <origin xyz="0 0 ${j1_length-base_height}" rpy="${pi/2} 0 0"/>
       <limit effort="6.0" lower="${-pi*(170/180)}" upper="${pi*(170/180)}" velocity="1.5708"/>
       <dynamics damping="1.0" friction="1.0"/>
@@ -221,5 +235,5 @@
       <child link="biorob_link3"/>
       <axis xyz="0 0 1 "/>
-      <origin xyz="${j2_length} 0 0.0"/>
+      <origin xyz="0 ${j2_length} 0" rpy="0 0 ${pi/2}"/>
       <limit effort="6.0" lower="${-pi*(100/180)}" upper="${pi*(100/180)}" velocity="1.5708"/>
       <dynamics damping="1.0" friction="1.0"/>
@@ -229,5 +243,5 @@
       <child link="biorob_link4"/>
       <axis xyz="0 0 1"/>
-      <origin xyz="${j3_length} 0 0.0"/>
+      <origin xyz="${j3_length} 0 0"/>
       <limit effort="6.0" lower="${-pi*(100/180)}" upper="${pi*(100/180)}" velocity="1.5708"/>
       <!-- TODO: give correct effort limits -->
@@ -245,6 +259,6 @@
       <parent link="biorob_link4"/>
       <child link="biorob_link5"/>
-      <axis xyz="1 0 0"/>
-      <origin xyz="${j5_length} 0.0 0 "/>
+      <axis xyz="0 0 1"/>
+      <origin xyz="${j5_length} 0 0" rpy="${pi/2} 0 ${pi/2}"/>
       <limit effort="6.0" lower="${-pi*(100/180)}" upper="${pi*(100/180)}" velocity="1.5708"/>
       <!-- TODO: give correct effort limits -->
@@ -255,5 +269,5 @@
       <child link="biorob_toolframe"/>
       <axis xyz="0 0 1"/>
-      <origin xyz="${j6_length} 0.0 0.0" rpy="${-pi/2} 0 0"/>
+      <origin xyz="0 0 ${j6_length}" rpy="0 0 0"/>
     </joint>
     <transmission type="pr2_mechanism_model/SimpleTransmission" name="joint1_trans">

File: fuerte/trunk/biorob_common/biorob_description/urdf/biorob_ultra_x5_ug/biorob_ultra_x5_ug.urdf.xacro (robot description, xacro)
@@ -1,9 +1,9 @@
 <?xml version="1.0"?>
-<robot name="biorob_ultra_x5_hg"
+<robot name="biorob_ultra_x5_ug"
     xmlns:sensor="http://playerstage.sourceforge.net/gazebo/xmlschema/#sensor"
     xmlns:controller="http://playerstage.sourceforge.net/gazebo/xmlschema/#controller"
     xmlns:interface="http://playerstage.sourceforge.net/gazebo/xmlschema/#interface">
     <!-- Included URDF Files -->
-    <include filename="$(find biorob_description)/urdf/biorob_ultra_x5_hg/biorob_ultra_x5_hg_base.urdf.xacro" />
+    <include filename="$(find biorob_description)/urdf/biorob_ultra_x5_ug/biorob_ultra_x5_ug_base.urdf.xacro" />
     <link name="base">
       <inertial>
@@ -15,6 +15,6 @@
 	</inertial>
       </link>
-    <biorob_ultra_x5_hg_arm parent="base" >
+    <biorob_ultra_x5_ug_arm parent="base" >
         <origin xyz="0 0 0" rpy="0 0 0"/>
-    </biorob_ultra_x5_hg_arm>
+    </biorob_ultra_x5_ug_arm>
 </robot>

File: fuerte/trunk/biorob_common/biorob_description/urdf/biorob_ultra_x5_ug/biorob_ultra_x5_ug_base.urdf.xacro (robot description, xacro)
@@ -4,13 +4,13 @@
        xmlns:interface="http://playerstage.sourceforge.net/gazebo/xmlschema/#interface"
        xmlns:xacro="http://playerstage.sourceforge.net/gazebo/xmlschema/#interface"
-       name="biorob_ultra_x6">
+       name="biorob_ultra_x5_ug">
   <xacro:property name="base_height" value=".01"/>
   <xacro:property name="j1_length" value=".284"/>
   <!--0.285 to base plate-->
   <xacro:property name="j2_length" value=".305"/>
-  <xacro:property name="j3_length" value=".10"/>
+  <xacro:property name="j3_length" value=".100"/>
   <xacro:property name="j4_length" value=".205"/>
-  <xacro:property name="j5_length" value=".14"/>
-  <xacro:property name="j6_length" value=".08"/>
+  <xacro:property name="j5_length" value=".150"/>
+  <!--<xacro:property name="j6_length" value=".08"/>-->
   <xacro:property name="pi" value="3.1415926536"/>
   <xacro:macro name="default_inertial" params="mass">
@@ -21,5 +21,5 @@
     </inertial>
   </xacro:macro>
-  <macro name="biorob_ultra_x6_arm" params="parent *origin">
+  <macro name="biorob_ultra_x5_ug_arm" params="parent *origin">
     <link name="biorob_base_link">
       <visual>
@@ -126,5 +126,5 @@
         <geometry>
           <mesh filename="package://biorob_description/meshes/biorob_x6/biorob_v3_x6_link_4.dae"/>
-          <!--                    <cylinder radius="0.002" length="0.001" />-->
+          <!--<cylinder radius="0.02" length="${j4_length}" />-->
         </geometry>
         <origin xyz="0 0 0" rpy="0 0 0"/>
@@ -150,5 +150,5 @@
         <geometry>
           <mesh filename="package://biorob_description/meshes/biorob_common/biorob_link_4.dae"/>
-          <!--  <cylinder radius="0.02" length="${j4_length}" />-->
+          <!--<cylinder radius="0.002" length="0.001" />-->
         </geometry>
         <origin xyz="0 0 0" rpy="${pi/2} 0 0"/>
@@ -159,5 +159,5 @@
         <geometry>
           <mesh filename="package://biorob_description/meshes/biorob_common/biorob_link_4.dae"/>
-          <!--<cylinder radius="0.02" length="${j4_length}" />-->
+          <!--<cylinder radius="0.002" length="0.001" />-->
         </geometry>
         <origin xyz="0 0 0" rpy="${pi/2} 0 0"/>
@@ -170,28 +170,4 @@
       <!--<material>HLUGV/Green</material>-->
     </gazebo>
-    <link name="biorob_link6">
-      <visual>
-        <geometry>
-          <mesh filename="package://biorob_description/meshes/biorob_ultra/biorob_ultra_tcp_end_80.dae"/>
-          <!--<cylinder radius="0.002" length="0.001" />-->
-        </geometry>
-        <origin xyz="0 0 0" rpy="0 0 0"/>
-        <material name="red">
-                </material>
-      </visual>
-      <collision>
-        <geometry>
-          <mesh filename="package://biorob_description/meshes/biorob_ultra/biorob_ultra_tcp_end_80.dae"/>
-          <!--<cylinder radius="0.002" length="0.001" />-->
-        </geometry>
-        <origin xyz="0 0 0" rpy="0 0 0"/>
-      </collision>
-      <xacro:default_inertial mass="0.01"/>
-    </link>
-    <gazebo reference="biorob_link6">
-      <selfCollide>true</selfCollide>
-      <material>biorob_material/Grey</material>
-      <!--<material>HLUGV/Green</material>-->
-    </gazebo>
     <link name="biorob_toolframe">
       <visual>
@@ -199,5 +175,5 @@
           <cylinder radius="0.01" length="0.001" />
         </geometry>
-        <origin xyz="0 0 0" rpy="0 0 0"/>
+        <origin xyz="0 0 0" rpy="${pi/2} 0 ${pi/2}"/>
         <material name="red">
         </material>
@@ -207,5 +183,5 @@
           <cylinder radius="0.02" length="0.001" />
         </geometry>
-        <origin xyz="0 0 0" rpy="0 0 0"/>
+        <origin xyz="0 0 0" rpy="${pi/2} 0 ${pi/2}"/>
       </collision>
       <xacro:default_inertial mass="0.05"/>
@@ -236,5 +212,5 @@
       <parent link="biorob_link2"/>
       <child link="biorob_link3"/>
-      <axis xyz="0 0 1 "/>
+      <axis xyz="0 0 1"/>
       <origin xyz="0 ${j2_length} 0" rpy="0 0 ${pi/2}"/>
       <limit effort="6.0" lower="${-pi*(100/180)}" upper="${pi*(100/180)}" velocity="1.5708"/>
@@ -245,5 +221,5 @@
       <child link="biorob_link4"/>
       <axis xyz="0 0 1"/>
-      <origin xyz="${j3_length} 0 0.0" rpy="${pi/2} 0 ${pi/2}"/>
+      <origin xyz="${j3_length} 0 0" rpy="${pi/2} 0 ${pi/2}"/>
       <limit effort="6.0" lower="${-pi*(100/180)}" upper="${pi*(100/180)}" velocity="1.5708"/>
       <!-- TODO: give correct effort limits -->
@@ -259,18 +235,9 @@
       <dynamics damping="1.0" friction="1.0"/>
     </joint>
-    <joint name="joint6" type="revolute">
+    <joint name="tool_frame" type="fixed">
       <parent link="biorob_link5"/>
-      <child link="biorob_link6"/>
-      <axis xyz="0 0 1"/>
-      <origin xyz="0 ${-j5_length} 0 " rpy="${pi/2} 0 0"/>
-      <limit effort="6.0" lower="${-pi*(100/180)}" upper="${pi*(100/180)}" velocity="1.5708"/>
-      <!-- TODO: give correct effort limits -->
-      <dynamics damping="1.0" friction="1.0"/>
-    </joint>
-    <joint name="tool_frame" type="fixed">
-      <parent link="biorob_link6"/>
       <child link="biorob_toolframe"/>
       <axis xyz="0 0 1"/>
-      <origin xyz="0 0 ${j6_length}" rpy="0 0 0"/>
+      <origin xyz="0 ${-j5_length} 0" rpy="0 0 ${-pi/2}"/>
     </joint>
     <transmission type="pr2_mechanism_model/SimpleTransmission" name="joint1_trans">

File: fuerte/trunk/biorob_common/biorob_description/urdf/biorob_v3_x4/biorob_v3_x4_base.urdf.xacro (robot description, xacro)
@@ -77,5 +77,5 @@
         </geometry>
         <!--<origin xyz="${j2_length/2 - j2_overhang_rear/2 } 0 0" rpy="0 ${pi/2} 0"/>-->
-        <origin xyz="0 0 0" rpy="${-pi/2} ${pi/2} 0"/>
+        <origin xyz="0 0 0" rpy="0 ${pi/2} ${pi}"/>
         <material name="red">
           <color rgba="0.6 0.6 0.6 1"/>
@@ -87,5 +87,5 @@
           <!--<cylinder radius="0.02" length="${j2_length}" />-->
         </geometry>
-        <origin xyz="0 0 0" rpy="${-pi/2} ${pi/2} 0"/>
+        <origin xyz="0 0 0" rpy="0 ${pi/2} ${pi}"/>
       </collision>
       <xacro:default_inertial mass="0.5"/>
@@ -145,4 +145,18 @@
     </gazebo>
     <link name="biorob_toolframe">
+      <visual>
+        <geometry>
+          <cylinder radius="0.01" length="0.001" />
+        </geometry>
+        <origin xyz="0 0 0" rpy="${pi/2} 0 ${pi/2}"/>
+        <material name="red">
+        </material>
+      </visual>
+      <collision>
+        <geometry>
+          <cylinder radius="0.02" length="0.001" />
+        </geometry>
+        <origin xyz="0 0 0" rpy="${pi/2} 0 ${pi/2}"/>
+      </collision>
       <xacro:default_inertial mass="0.05"/>
     </link>
@@ -165,5 +179,5 @@
       <child link="biorob_link2"/>
       <axis xyz="0 0 1"/>
-      <origin xyz="0 0 ${j1_length-base_height}" rpy="${pi/2} -${pi/2} 0"/>
+      <origin xyz="0 0 ${j1_length-base_height}" rpy="${pi/2} 0 0"/>
       <limit effort="6.0" lower="${-pi*(170/180)}" upper="${pi*(170/180)}" velocity="1.5708"/>
       <dynamics damping="1.0" friction="1.0"/>
@@ -173,5 +187,5 @@
       <child link="biorob_link3"/>
       <axis xyz="0 0 1 "/>
-      <origin xyz="${j2_length} 0 0.0"/>
+      <origin xyz="0 ${j2_length} 0" rpy="0 0 ${pi/2}"/>
       <limit effort="6.0" lower="${-pi*(100/180)}" upper="${pi*(100/180)}" velocity="1.5708"/>
       <dynamics damping="1.0" friction="1.0"/>
@@ -190,5 +204,5 @@
       <child link="biorob_toolframe"/>
       <axis xyz="0 0 1"/>
-      <origin xyz="${j4_length} 0.0 0.0" rpy="${-pi/2} 0 0"/>
+      <origin xyz="${j4_length} 0.0 0.0" rpy="0 0 0"/>
     </joint>
     <transmission type="pr2_mechanism_model/SimpleTransmission" name="joint1_trans">
