Commit message: [hlugv_description] -add proper color to wheels in fuerte -increase wheel weight

File: fuerte/trunk/hlugv_common/hlugv_description/urdf/hlugv_wheel.urdf.xacro (robot description, xacro)
@@ -26,5 +26,5 @@
         <link name="${prefix}_wheel_link">
             <inertial>
-                <mass value="0.1" />
+                <mass value="0.2" />
                 <origin xyz=" 0 0 0 " />
                 <inertia  ixx="0.00012411765597" ixy="0.0" ixz="0.0"
@@ -54,5 +54,5 @@
             <kp  value="100000.0" />
             <kd  value="1.0" />
-            <material>HLUGV/Grey</material>
+	    <material>Gazebo/Grey</material>
         </gazebo>
         <transmission type="pr2_mechanism_model/SimpleTransmission" name="${prefix}_wheel_trans">
