Commit message: merged from /trunk/hector_quadrotor

File: branches/gazebo-1.5/hector_quadrotor/hector_quadrotor_controller/urdf/quadrotor_controller.urdf.xacro (robot description, xacro)
@@ -1,11 +1,8 @@
 <?xml version="1.0"?>
-<robot
-xmlns:controller="http://playerstage.sourceforge.net/gazebo/xmlschema/#controller"
-xmlns:xacro="http://ros.org/wiki/xacro"
->
+<robot xmlns:xacro="http://ros.org/wiki/xacro">
   <!-- Quadrotor Controller Plugin -->
   <xacro:macro name="quadrotor_controller" params="state_topic imu_topic">
     <gazebo>
-      <controller:hector_quadrotor_controller name="quadrotor_controller" plugin="libhector_quadrotor_controller.so">
+      <plugin name="quadrotor_controller" filename="libgazebo_rtt_plugin.so">
         <updateRate>100.0</updateRate>
         <import>quadro</import>
@@ -19,5 +16,5 @@
         <port name="motor_output" topic="motor_pwm" queue_size="10" />
         <port name="height" />
-      </controller:hector_quadrotor_controller>
+      </plugin>
     </gazebo>
   </xacro:macro>

File: branches/gazebo-1.5/hector_quadrotor/hector_quadrotor_controller/urdf/quadrotor_pose_estimation.urdf.xacro (robot description, xacro)
@@ -4,8 +4,8 @@
 xmlns:xacro="http://ros.org/wiki/xacro"
 >
-  <!-- Quadrotor Controller Plugin -->
-  <xacro:macro name="quadrotor_controller" params="state_topic imu_topic">
+  <!-- Quadrotor Pose Estimation Plugin -->
+  <xacro:macro name="quadrotor_pose_estimation">
     <gazebo>
-      <controller:hector_quadrotor_pose_estimation name="quadrotor_pose_estimation" plugin="libgazebo_rtt_plugin.so">
+      <plugin name="quadrotor_pose_estimation" filename="libgazebo_rtt_plugin.so">
         <updateRate>100.0</updateRate>
         <import>hector_pose_estimation_rtt</import>
@@ -18,20 +18,5 @@
         <port name="state" queue_size="10" />
         <port name="imu" queue_size="10" />
-      </controller:hector_quadrotor_pose_estimation>
-      <controller:mbn name="model_based_navigation" plugin="libgazebo_rtt_plugin.so">
-        <updateRate>100.0</updateRate>
-        <import>quadro</import>
-        <component>Simulink</component>
-        <property name="Model">$(find quadro)/simulink/MBN/RTWmodel_QK_SFSVD_ROS.so</property>
-        <port name="raw_imu" queue_size="10" />
-        <port name="magnetic" />
-        <port name="altimeter" />
-        <port name="fix" />
-        <port name="fix_velocity" />
-        <port name="motor_status" />
-        <port name="state" topic="mbn/state" queue_size="10" />
-        <port name="imu" topic="mbn/imu" queue_size="10" />
-        <port name="log" topic="mbn/log" queue_size="10" />
-      </controller:mbn>
+      </plugin>
     </gazebo>
   </xacro:macro>
